File: ergodox_extended.kicad_pro.kicad_pcb (KiCad board)
At the start: 2 copper layers, 201.9 x 170.2 mm, 129 parts, among them J1 USB_B_Micro, J2 AudioJack4, J3 AudioJack4, J4 ISP, SW0:0 SWITCH, SW0:1 SWITCH, SW0:2 SWITCH, SW0:3 SWITCH, SW0:4 SWITCH, SW0:5 SWITCH, SW0:6 SWITCH, SW1 Reset, SW1:0 SWITCH, SW1:1 SWITCH, SW1:2 SWITCH, SW1:3 SWITCH, SW1:4 SWITCH, SW1:5 SWITCH, SW1:6 SWITCH, SW2:0 SWITCH, SW2:1 SWITCH, SW2:2 SWITCH, SW2:3 SWITCH, SW2:4 SWITCH, SW2:5 SWITCH, SW2:6 SWITCH, SW3:0 SWITCH, SW3:1 SWITCH, SW3:2 SWITCH, SW3:3 SWITCH, SW3:4 SWITCH, SW3:5 SWITCH, SW3:6 SWITCH, SW4:0 SWITCH, SW4:1 SWITCH, SW4:2 SWITCH, SW4:3 SWITCH, SW4:4 SWITCH, SW4:5 SWITCH, SW4:6 SWITCH, SW5:0 SWITCH, SW5:1 SWITCH, SW5:2 SWITCH, SW5:3 SWITCH, SW5:4 SWITCH, SW5:5 SWITCH, SW5:6 SWITCH, SW6:0 SWITCH, SW6:1 SWITCH, SW6:2 SWITCH, SW6:3 SWITCH, SW6:4 SWITCH, SW6:5 SWITCH, SW6:6 SWITCH, U1 ATmega32U4-AU, U2 MCP23018-E_SS, Y1 16Mhz

Commit message: Fix diode dir, write readme
Parts:
- turned D0:0 to -60 degrees
- turned D0:1 to -60 degrees
- turned D0:2 to -150 degrees
- turned D0:3 to -60 degrees
- turned D0:4 to -60 degrees
- turned D0:5 to -60 degrees
- turned D0:6 to -60 degrees
- turned D1:0 to -90 degrees
- turned D1:1 to -90 degrees
- turned D1:2 to -90 degrees
- turned D1:3 to -90 degrees
- turned D1:4 to -90 degrees
- turned D1:5 to 120 degrees
- turned D1:6 to -150 degrees
- turned D2:0 to -90 degrees
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Connections:
- D0:0 pad 1: Col0 -> Net-(D0:0-K)
- D0:0 pad 2: Net-(D0:0-Pad2) -> Col0
- D0:1 pad 1: Col1 -> Net-(D0:1-K)
- D0:1 pad 2: Net-(D0:1-Pad2) -> Col1
- D0:2 pad 1: Col2 -> Net-(D0:2-K)
- D0:2 pad 2: Net-(D0:2-Pad2) -> Col2
- D0:3 pad 1: Col3 -> Net-(D0:3-K)
- D0:3 pad 2: Net-(D0:3-Pad2) -> Col3
- D0:4 pad 1: Col4 -> Net-(D0:4-K)
- D0:4 pad 2: Net-(D0:4-Pad2) -> Col4
- D0:5 pad 1: Col5 -> Net-(D0:5-K)
- D0:5 pad 2: Net-(D0:5-Pad2) -> Col5
- D0:6 pad 1: Col6 -> Net-(D0:6-K)
- D0:6 pad 2: Net-(D0:6-Pad2) -> Col6
- D1:0 pad 1: Col0 -> Net-(D1:0-K)
- D1:0 pad 2: Net-(D1:0-Pad2) -> Col0
- D1:1 pad 1: Col1 -> Net-(D1:1-K)
- D1:1 pad 2: Net-(D1:1-Pad2) -> Col1
- D1:2 pad 1: Col2 -> Net-(D1:2-K)
- D1:2 pad 2: Net-(D1:2-Pad2) -> Col2
- D1:3 pad 1: Col3 -> Net-(D1:3-K)
- D1:3 pad 2: Net-(D1:3-Pad2) -> Col3
- D1:4 pad 1: Col4 -> Net-(D1:4-K)
- D1:4 pad 2: Net-(D1:4-Pad2) -> Col4
- D1:5 pad 1: Col5 -> Net-(D1:5-K)
- D1:5 pad 2: Net-(D1:5-Pad2) -> Col5
- D1:6 pad 1: Col6 -> Net-(D1:6-K)
- D1:6 pad 2: Net-(D1:6-Pad2) -> Col6
- D2:0 pad 1: Col0 -> Net-(D2:0-K)
- D2:0 pad 2: Net-(D2:0-Pad2) -> Col0
- D2:1 pad 1: Col1 -> Net-(D2:1-K)
- D2:1 pad 2: Net-(D2:1-Pad2) -> Col1
- D2:2 pad 1: Col2 -> Net-(D2:2-K)
- D2:2 pad 2: Net-(D2:2-Pad2) -> Col2
- D2:3 pad 1: Col3 -> Net-(D2:3-K)
- D2:3 pad 2: Net-(D2:3-Pad2) -> Col3
- D2:4 pad 1: Col4 -> Net-(D2:4-K)
- D2:4 pad 2: Net-(D2:4-Pad2) -> Col4
- D2:5 pad 1: Col5 -> Net-(D2:5-K)
- D2:5 pad 2: Net-(D2:5-Pad2) -> Col5
- D2:6 pad 1: Col6 -> Net-(D2:6-K)
- D2:6 pad 2: Net-(D2:6-Pad2) -> Col6
- D3:0 pad 1: Col0 -> Net-(D3:0-K)
- D3:0 pad 2: Net-(D3:0-Pad2) -> Col0
- D3:1 pad 1: Col1 -> Net-(D3:1-K)
- D3:1 pad 2: Net-(D3:1-Pad2) -> Col1
- D3:2 pad 1: Col2 -> Net-(D3:2-K)
- D3:2 pad 2: Net-(D3:2-Pad2) -> Col2
- D3:3 pad 1: Col3 -> Net-(D3:3-K)
- D3:3 pad 2: Net-(D3:3-Pad2) -> Col3
- D3:4 pad 1: Col4 -> Net-(D3:4-K)
- D3:4 pad 2: Net-(D3:4-Pad2) -> Col4
- D3:5 pad 1: Col5 -> Net-(D3:5-K)
- D3:5 pad 2: Net-(D3:5-Pad2) -> Col5
- D3:6 pad 1: Col6 -> Net-(D3:6-K)
- D3:6 pad 2: Net-(D3:6-Pad2) -> Col6
- D4:0 pad 1: Col0 -> Net-(D4:0-K)
- D4:0 pad 2: Net-(D4:0-Pad2) -> Col0
- D4:1 pad 1: Col1 -> Net-(D4:1-K)
- D4:1 pad 2: Net-(D4:1-Pad2) -> Col1
- D4:2 pad 1: Col2 -> Net-(D4:2-K)
- D4:2 pad 2: Net-(D4:2-Pad2) -> Col2
- D4:3 pad 1: Col3 -> Net-(D4:3-K)
- D4:3 pad 2: Net-(D4:3-Pad2) -> Col3
- D4:4 pad 1: Col4 -> Net-(D4:4-K)
- D4:4 pad 2: Net-(D4:4-Pad2) -> Col4
- D4:5 pad 1: Col5 -> Net-(D4:5-K)
- D4:5 pad 2: Net-(D4:5-Pad2) -> Col5
- D4:6 pad 1: Col6 -> Net-(D4:6-K)
- D4:6 pad 2: Net-(D4:6-Pad2) -> Col6
- D5:0 pad 1: Col0 -> Net-(D5:0-K)
- D5:0 pad 2: Net-(D5:0-Pad2) -> Col0
- D5:1 pad 1: Col1 -> Net-(D5:1-K)
- D5:1 pad 2: Net-(D5:1-Pad2) -> Col1
- D5:2 pad 1: Col2 -> Net-(D5:2-K)
- D5:2 pad 2: Net-(D5:2-Pad2) -> Col2
- D5:3 pad 1: Col3 -> Net-(D5:3-K)
- D5:3 pad 2: Net-(D5:3-Pad2) -> Col3
- D5:4 pad 1: Col4 -> Net-(D5:4-K)
- D5:4 pad 2: Net-(D5:4-Pad2) -> Col4
- D5:5 pad 1: Col5 -> Net-(D5:5-K)
- D5:5 pad 2: Net-(D5:5-Pad2) -> Col5
- D5:6 pad 1: Col6 -> Net-(D5:6-K)
- D5:6 pad 2: Net-(D5:6-Pad2) -> Col6
- D6:0 pad 1: Col0 -> Net-(D6:0-K)
- D6:0 pad 2: Net-(D6:0-Pad2) -> Col0
- D6:1 pad 1: Col1 -> Net-(D6:1-K)
- D6:1 pad 2: Net-(D6:1-Pad2) -> Col1
- D6:2 pad 1: Col2 -> Net-(D6:2-K)
- D6:2 pad 2: Net-(D6:2-Pad2) -> Col2
- D6:3 pad 1: Col3 -> Net-(D6:3-K)
- D6:3 pad 2: Net-(D6:3-Pad2) -> Col3
- D6:4 pad 1: Col4 -> Net-(D6:4-K)
- D6:4 pad 2: Net-(D6:4-Pad2) -> Col4
- D6:5 pad 1: Col5 -> Net-(D6:5-K)
- D6:5 pad 2: Net-(D6:5-Pad2) -> Col5
- D6:6 pad 1: Col6 -> Net-(D6:6-K)
- D6:6 pad 2: Net-(D6:6-Pad2) -> Col6
- SW0:0 pad 2: Net-(D0:0-Pad2) -> Net-(D0:0-K)
- SW0:1 pad 2: Net-(D0:1-Pad2) -> Net-(D0:1-K)
- SW0:2 pad 2: Net-(D0:2-Pad2) -> Net-(D0:2-K)
- SW0:3 pad 2: Net-(D0:3-Pad2) -> Net-(D0:3-K)
- SW0:4 pad 2: Net-(D0:4-Pad2) -> Net-(D0:4-K)
- SW0:5 pad 2: Net-(D0:5-Pad2) -> Net-(D0:5-K)
- SW0:6 pad 2: Net-(D0:6-Pad2) -> Net-(D0:6-K)
- SW1:0 pad 2: Net-(D1:0-Pad2) -> Net-(D1:0-K)
- SW1:1 pad 2: Net-(D1:1-Pad2) -> Net-(D1:1-K)
- SW1:2 pad 2: Net-(D1:2-Pad2) -> Net-(D1:2-K)
- SW1:3 pad 2: Net-(D1:3-Pad2) -> Net-(D1:3-K)
- SW1:4 pad 2: Net-(D1:4-Pad2) -> Net-(D1:4-K)
- SW1:5 pad 2: Net-(D1:5-Pad2) -> Net-(D1:5-K)
- SW1:6 pad 2: Net-(D1:6-Pad2) -> Net-(D1:6-K)
- SW2:0 pad 2: Net-(D2:0-Pad2) -> Net-(D2:0-K)
- SW2:1 pad 2: Net-(D2:1-Pad2) -> Net-(D2:1-K)
- SW2:2 pad 2: Net-(D2:2-Pad2) -> Net-(D2:2-K)
- SW2:3 pad 2: Net-(D2:3-Pad2) -> Net-(D2:3-K)
- SW2:4 pad 2: Net-(D2:4-Pad2) -> Net-(D2:4-K)
- SW2:5 pad 2: Net-(D2:5-Pad2) -> Net-(D2:5-K)
- SW2:6 pad 2: Net-(D2:6-Pad2) -> Net-(D2:6-K)
- SW3:0 pad 2: Net-(D3:0-Pad2) -> Net-(D3:0-K)
- SW3:1 pad 2: Net-(D3:1-Pad2) -> Net-(D3:1-K)
- SW3:2 pad 2: Net-(D3:2-Pad2) -> Net-(D3:2-K)
- SW3:3 pad 2: Net-(D3:3-Pad2) -> Net-(D3:3-K)
- SW3:4 pad 2: Net-(D3:4-Pad2) -> Net-(D3:4-K)
- SW3:5 pad 2: Net-(D3:5-Pad2) -> Net-(D3:5-K)
- SW3:6 pad 2: Net-(D3:6-Pad2) -> Net-(D3:6-K)
- SW4:0 pad 2: Net-(D4:0-Pad2) -> Net-(D4:0-K)
- SW4:1 pad 2: Net-(D4:1-Pad2) -> Net-(D4:1-K)
- SW4:2 pad 2: Net-(D4:2-Pad2) -> Net-(D4:2-K)
- SW4:3 pad 2: Net-(D4:3-Pad2) -> Net-(D4:3-K)
- SW4:4 pad 2: Net-(D4:4-Pad2) -> Net-(D4:4-K)
- SW4:5 pad 2: Net-(D4:5-Pad2) -> Net-(D4:5-K)
- SW4:6 pad 2: Net-(D4:6-Pad2) -> Net-(D4:6-K)
- SW5:0 pad 2: Net-(D5:0-Pad2) -> Net-(D5:0-K)
- SW5:1 pad 2: Net-(D5:1-Pad2) -> Net-(D5:1-K)
- SW5:2 pad 2: Net-(D5:2-Pad2) -> Net-(D5:2-K)
- SW5:3 pad 2: Net-(D5:3-Pad2) -> Net-(D5:3-K)
- SW5:4 pad 2: Net-(D5:4-Pad2) -> Net-(D5:4-K)
- SW5:5 pad 2: Net-(D5:5-Pad2) -> Net-(D5:5-K)
- SW5:6 pad 2: Net-(D5:6-Pad2) -> Net-(D5:6-K)
- SW6:0 pad 2: Net-(D6:0-Pad2) -> Net-(D6:0-K)
- SW6:1 pad 2: Net-(D6:1-Pad2) -> Net-(D6:1-K)
- SW6:2 pad 2: Net-(D6:2-Pad2) -> Net-(D6:2-K)
- SW6:3 pad 2: Net-(D6:3-Pad2) -> Net-(D6:3-K)
- SW6:4 pad 2: Net-(D6:4-Pad2) -> Net-(D6:4-K)
- SW6:5 pad 2: Net-(D6:5-Pad2) -> Net-(D6:5-K)
- SW6:6 pad 2: Net-(D6:6-Pad2) -> Net-(D6:6-K)
Routing:
- net Net-(D1:6-Pad2): track 19.7 -> 0.00 mm
- net Net-(D1:6-K): track 0.00 -> 19.7 mm
- net Net-(D2:6-Pad2): track 19.5 -> 0.00 mm
- net Net-(D2:6-K): track 0.00 -> 19.5 mm
- net Net-(D1:5-Pad2): track 19.5 -> 0.00 mm
- net Net-(D1:5-K): track 0.00 -> 19.5 mm
- net Net-(D3:6-Pad2): track 12.8 -> 0.00 mm
- net Net-(D3:6-K): track 0.00 -> 12.8 mm
- net Net-(D4:4-Pad2): track 12.6 -> 0.00 mm
- net Net-(D4:4-K): track 0.00 -> 12.6 mm
- net Net-(D3:4-Pad2): track 12.6 -> 0.00 mm
- net Net-(D3:4-K): track 0.00 -> 12.6 mm
- net Net-(D2:4-Pad2): track 12.6 -> 0.00 mm
- net Net-(D2:4-K): track 0.00 -> 12.6 mm
- net Net-(D5:4-Pad2): track 12.6 -> 0.00 mm
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Other:
- board text added: "Version 2.2 2024.03.24"
- board text removed: "Version 2.1 2024.03.13"
